Commit message: Created joint for robot

File: description/robot_core.xacro (robot description, xacro)
@@ -1,3 +1,30 @@
 <?xml version="1.0"?>
 <robot xmlns:xacro="http://www.ros.org/wiki/xacro">
+    <material name="white">
+        <color rgba="1 1 1 1" />
+    </material>
+    <material name="orange">
+        <color rgba="1 0.3 0.1 1" />
+    </material>
+    <material name="blue">
+        <color rgba="0.2 0.2 1 1" />
+    </material>
+    <material name="black">
+        <color rgba="0 0 0 1" />
+    </material>
+    <link name="base_link">
+    </link>
+    <joint name="chassis_joint" type="fixed">
+        <parent link="base_link"/>
+        <child link="chassis"/>
+        <origin xyz="-0.1 0 0"/>
+    </joint>
+    <link name="chassis">
+        <visual>
+            <origin xyz="0.15 0 0.075"/>
+            <geometry>
+                <box size="0.3 0.3 0.15"/>
+            </geometry>
+            <material name="white"/>
+        </visual>
 </robot>

Commit message: Made model look similar to real robot

File: description/robot_core.xacro (robot description, xacro)
@@ -13,6 +13,8 @@
         <color rgba="0 0 0 1" />
     </material>
+    <!-- BASE LINK -->
     <link name="base_link">
     </link>
+    <!-- CHASSIS LINK -->
     <joint name="chassis_joint" type="fixed">
         <parent link="base_link"/>
@@ -22,9 +24,40 @@
     <link name="chassis">
         <visual>
-            <origin xyz="0.15 0 0.075"/>
+            <origin xyz="0.381 0 0.09"/>
             <geometry>
-                <box size="0.3 0.3 0.15"/>
+                <cylinder radius="0.381" length="0.115"/>
             </geometry>
-            <material name="white"/>
+            <material name="orange"/>
         </visual>
+    <link/>
+    <!-- LEFT WHEEL LINK -->
+    <joint name="left_wheel_joint" type="continuous">
+        <parent link="base_link"/>
+        <child link="left_wheel"/>
+        <origin xyz="0 0.145 0" rpy="-${pi/2} 0 0"/>
+        <axis xyz="0 0 1"/>
+    </joint>
+    <link name="left_wheel">
+        <visual>
+            <geometry>
+                <cylinder radius="0.0635" length="0.0508"/>
+            </geometry>
+            <material name="blue">
+        </visual>
+    </link>
+    <!-- RIGHT WHEEL LINK -->
+    <joint name="left_right_joint" type="continuous">
+        <parent link="base_link"/>
+        <child link="right_wheel"/>
+        <origin xyz="0 -0.145 0" rpy="${pi/2} 0 0"/>
+        <axis xyz="0 0 -1"/>
+    </joint>
+    <link name="right_wheel">
+        <visual>
+            <geometry>
+                <cylinder radius="0.0635" length="0.04"/>
+            </geometry>
+            <material name="blue">
+        </visual>
+    </link>
 </robot>

Commit message: Testing GIt

File: description/robot_core.xacro (robot description, xacro)
@@ -35,5 +35,5 @@
     <parent link="base_link"/>
     <child link="left_wheel"/>
-    <origin xyz="0 0.145 0" rpy="-${pi/2} 0 0"/>
+    <origin xyz="0.25 0.2 0" rpy="-${pi/2} 0 0"/>
     <axis xyz="0 0 1"/>
   </joint>
@@ -41,5 +41,5 @@
     <visual>
       <geometry>
-        <cylinder radius="0.0635" length="0.0508"/>
+        <cylinder radius="0.08" length="0.0508"/>
       </geometry>
       <material name="blue"/>
@@ -50,5 +50,5 @@
     <parent link="base_link"/>
     <child link="right_wheel"/>
-    <origin xyz="0 -0.145 0" rpy="${pi/2} 0 0"/>
+    <origin xyz="0.25 -0.2 0" rpy="${pi/2} 0 0"/>
     <axis xyz="0 0 -1"/>
   </joint>
@@ -56,5 +56,5 @@
     <visual>
       <geometry>
-        <cylinder radius="0.0635" length="0.04"/>
+        <cylinder radius="0.08" length="0.0508"/>
       </geometry>
       <material name="blue"/>

Commit message: Added The Caster Wheel Link

File: description/robot_core.xacro (robot description, xacro)
@@ -1,4 +1,4 @@
 <?xml version="1.0"?>
-<robot xmlns:xacro="http://ros.org/wiki/xacro">
+<robot xmlns:xacro="http://www.ros.org/wiki/xacro" name="robot">
   <!-- Materials -->
   <material name="white">
@@ -16,5 +16,5 @@
   <!-- Base Link -->
   <link name="base_link"/>
-  <!-- Chassis -->
+  <!-- Chassis Link -->
   <joint name="chassis_joint" type="fixed">
     <parent link="base_link"/>
@@ -31,5 +31,5 @@
     </visual>
   </link>
-  <!-- Left Wheel -->
+  <!-- Left Wheel Link -->
   <joint name="left_wheel_joint" type="continuous">
     <parent link="base_link"/>
@@ -46,5 +46,5 @@
     </visual>
   </link>
-  <!-- Right Wheel -->
+  <!-- Right Wheel Link -->
   <joint name="right_wheel_joint" type="continuous">
     <parent link="base_link"/>
@@ -61,3 +61,17 @@
     </visual>
   </link>
+  <!-- Caster Wheel Link -->
+  <joint name="caster_wheel_joint" type="fixed">
+    <parent link="chassis"/>
+    <child link="caster_wheel"/>
+    <origin xyz="0.1 0 0"/>
+  </joint>
+  <link name="caster_wheel">
+    <visual>
+      <geometry>
+        <sphere radius="0.075"/>
+      </geometry>
+      <material name="black"/>
+    </visual>
+  </link>
 </robot>

Commit message: Added Collision for the robot *NEED TO TEST*

File: description/robot_core.xacro (robot description, xacro)
@@ -30,4 +30,10 @@
       <material name="orange"/>
     </visual>
+    <collision>
+      <origin xyz="0.381 0 0.09"/>
+      <geometry>
+        <cylinder radius="0.381" length="0.115"/>
+      </geometry>
+    </collision>
   </link>
   <!-- Left Wheel Link -->
@@ -45,4 +51,9 @@
       <material name="blue"/>
     </visual>
+    <collision>
+      <geometry>
+        <cylinder radius="0.08" length="0.0508"/>
+      </geometry>
+    </collision>
   </link>
   <!-- Right Wheel Link -->
@@ -60,4 +71,9 @@
       <material name="blue"/>
     </visual>
+    <collision>
+      <geometry>
+        <cylinder radius="0.08" length="0.0508"/>
+      </geometry>
+    </collision>
   </link>
   <!-- Caster Wheel Link -->
@@ -74,4 +90,9 @@
       <material name="black"/>
     </visual>
+    <collision>
+      <geometry>
+        <sphere radius="0.075"/>
+      </geometry>
+    </collision>
   </link>
 </robot>

Commit message: Added inertial_macros.xacro file and added the macro into the robot_core.xacro

File: description/robot_core.xacro (robot description, xacro)
@@ -1,4 +1,5 @@
 <?xml version="1.0"?>
 <robot xmlns:xacro="http://www.ros.org/wiki/xacro" name="robot">
+  <xacro:include filename="inertial_macros.xacro"/>
   <!-- Materials -->
   <material name="white">
@@ -36,4 +37,7 @@
       </geometry>
     </collision>
+    <xacro:inertial_cylinder mass="0.5" radius="0.381" length="0.115"/>
+        <origin xyz="0.381 0 0.09" rpy="0 0 0"/>
+    </xacro:inertial_cylinder>
   </link>
   <!-- Left Wheel Link -->
@@ -56,4 +60,7 @@
       </geometry>
     </collision>
+    <xacro:inertial_cylinder mass="0.1" length="0.0508" radius="0.08"/>
+        <origin xyz="0 0 0" rpy="0 0 0"/>
+    </xacro:inertial_cylinder>
   </link>
   <!-- Right Wheel Link -->
@@ -76,4 +83,7 @@
       </geometry>
     </collision>
+    <xacro:inertial_cylinder mass="0.1" length="0.0508" radius="0.08"/>
+        <origin xyz="0 0 0" rpy="0 0 0"/>
+    </xacro:inertial_cylinder>
   </link>
   <!-- Caster Wheel Link -->
@@ -95,4 +105,7 @@
       </geometry>
     </collision>
+    <inertial_sphere mass="0.1" radius="0.075"/>
+        <origin xyz="0 0 0" rpy="0 0 0"/>
+    </inertial_sphere>
   </link>
 </robot>
